Commit message: Major IK and URDF Updates

File: Teleoperation/ur10.urdf (robot description, URDF)
Before this commit: robot ur10_from_dh, 9 links, 8 joints
Links:
- link base_link: geometry visual cylinder length=0.05 radius=0.15
- link link1: geometry visual cylinder length=0.05 radius=0.10
- link link2: geometry visual cylinder length=0.400 radius=0.06
- link link3: geometry visual sphere radius=0.07
- link link4: geometry visual cylinder length=0.2605 radius=0.05
- link link5: geometry visual sphere radius=0.06
- link link6: geometry visual cylinder length=0.074 radius=0.04
- link tool0: geometry visual cylinder length=0.01 radius=0.05
Joints:
- joint joint1: limit lower=-6.28 upper=6.28 effort=150 velocity=3.14 -> lower=-2.094 upper=2.094 effort=300 velocity=3.14; origin xyz=0 0 7.47 rpy=-1.5708 0 0 -> xyz=0 0 0.150 rpy=0 0 0
- joint joint2: axis 0 0 1 -> 0 1 0; limit lower=-6.28 upper=6.28 effort=150 velocity=3.14 -> lower=-2.094 upper=2.094 effort=300 velocity=3.14; origin xyz=41 0 0 rpy=0 0 0 -> xyz=0 0 0.0449 rpy=0 0 0
- joint joint3: axis 0 0 1 -> 0 1 0; limit lower=-6.28 upper=6.28 effort=150 velocity=3.14 -> lower=-2.094 upper=2.094 effort=300 velocity=3.14; origin xyz=0.95 0 0 rpy=1.5708 0 0 -> xyz=0 0 0.400 rpy=0 0 0
- joint joint4: limit lower=-6.28 upper=6.28 effort=28 velocity=3.14 -> lower=-2.094 upper=2.094 effort=28 velocity=3.14; origin xyz=0 0 26.94 rpy=1.5708 0 0 -> xyz=0 0 0.0654 rpy=0 0 0
- joint joint5: axis 0 0 1 -> 0 1 0; limit lower=-6.28 upper=6.28 effort=28 velocity=3.14 -> lower=-2.094 upper=2.094 effort=28 velocity=3.14; origin xyz=0 0 3 rpy=-1.5708 0 0 -> xyz=0 0 0.2605 rpy=0 0 0
- joint joint6: limit lower=-6.28 upper=6.28 effort=28 velocity=3.14 -> lower=-2.094 upper=2.094 effort=28 velocity=3.14; origin xyz=0 0 20 rpy=0 0 0 -> xyz=0 0 0.071 rpy=0 0 0
- joint link6_to_tool0: origin xyz=0 0 0.20 rpy=0 0 0 -> xyz=0 0 0.074 rpy=0 0 0
- joint world_to_base: origin xyz=0 0 0 rpy=0 0 0 -> (none)

Commit message: significant refinements to latency and IK

File: Teleoperation/ur10.urdf (robot description, URDF)
Before this commit: robot my_robot, 9 links, 8 joints
Joints:
- joint joint1: limit lower=-2.094 upper=2.094 effort=300 velocity=3.14 -> lower=-2.094 upper=2.094 effort=300 velocity=3.142
- joint joint2: limit lower=-2.094 upper=2.094 effort=300 velocity=3.14 -> lower=-1.7 upper=1.7 effort=300 velocity=3.142
- joint joint3: limit lower=-2.094 upper=2.094 effort=300 velocity=3.14 -> lower=-2.094 upper=2.094 effort=300 velocity=3.142
- joint joint4: limit lower=-2.094 upper=2.094 effort=28 velocity=3.14 -> lower=-2.094 upper=2.094 effort=28 velocity=3.142
- joint joint5: limit lower=-2.094 upper=2.094 effort=28 velocity=3.14 -> lower=-2.094 upper=2.094 effort=28 velocity=3.142
- joint joint6: limit lower=-2.094 upper=2.094 effort=28 velocity=3.14 -> lower=-2.094 upper=2.094 effort=28 velocity=3.142

Commit message: quick change

File: Teleoperation/ur10.urdf (robot description, URDF)
Before this commit: robot my_robot, 9 links, 8 joints
Joints:
- joint joint1: limit lower=-2.094 upper=2.094 effort=300 velocity=3.142 -> lower=-2.094 upper=2.094 effort=300 velocity=25.136
- joint joint2: limit lower=-1.7 upper=1.7 effort=300 velocity=3.142 -> lower=-1.7 upper=1.7 effort=300 velocity=25.136
- joint joint3: limit lower=-2.094 upper=2.094 effort=300 velocity=3.142 -> lower=-2.094 upper=2.094 effort=300 velocity=25.136
- joint joint4: limit lower=-2.094 upper=2.094 effort=28 velocity=3.142 -> lower=-2.094 upper=2.094 effort=28 velocity=25.136
- joint joint5: limit lower=-2.094 upper=2.094 effort=28 velocity=3.142 -> lower=-2.094 upper=2.094 effort=28 velocity=25.136
- joint joint6: limit lower=-2.094 upper=2.094 effort=28 velocity=3.142 -> lower=-2.094 upper=2.094 effort=28 velocity=25.136

Commit message: control improvements and UI improvements

File: Teleoperation/ur10.urdf (robot description, URDF)
Before this commit: robot my_robot, 9 links, 8 joints
Joints:
- joint joint1: limit lower=-2.094 upper=2.094 effort=300 velocity=25.136 -> effort=300 velocity=25.136
- joint joint3: limit lower=-2.094 upper=2.094 effort=300 velocity=25.136 -> lower=-2.7 upper=2.7 effort=300 velocity=25.136
- joint joint4: limit lower=-2.094 upper=2.094 effort=28 velocity=25.136 -> lower=-3 upper=3 effort=28 velocity=25.136
